Commit message: New map for cartographer

File: description/lidar.xacro (robot description, xacro)
@@ -4,5 +4,5 @@
         <parent link="chassis"/>
         <child link="laser"/>
-        <origin xyz="0.1 0 0.515" rpy="0 0 0"/>
+        <origin xyz="0.1 0 0.515" rpy="0 0 -3.14"/>
     </joint>
     <link name="laser">
